File: RP2040 Dev Board.kicad_pcb (KiCad board)
At the start: 4 copper layers, 20.3 x 48.3 mm, 106 parts, among them J101 Conn_01x19, J102 Conn_01x19, J103 Conn_01x03, J201 TYPE-C-31-M-12, SW202 ~{USB_BOOT}, U201 AZ1117R-3.3TRE1, U202 RP2040, U205 W25Q128JVS, Y201 Crystal_GND24

Commit message: Added Prepreg JLC7628 Note
The dimensions for the differential USB lines were calculated based off the JLC7628 prepreg.
Other:
- board text added: "Controlled impedance USB traces designed for JLC7628 Prepreg."
Changed lines of the file:
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@@
   (title_block
     (title "RP2040 Template")
-    (date "2022-05-17")
+    (date "2022-05-18")
     (rev "4")
     (company "J & R Creative Technologies Inc.")
@@
     (effects (font (size 1 1) (thickness 0.15)) (justify mirror))
   )
+  (gr_text "Controlled impedance USB traces\ndesigned for JLC7628 Prepreg." (at 181.21 49.74) (layer "F.Fab")
+    (effects (font (size 1 1) (thickness 0.15)))
+  )
   (segment (start 146.64 54.62) (end 146.64 55.15) (width 0.2) (layer "F.Cu") (net 1))
